File: ModemHAT.kicad_pcb (KiCad board)
At the start: 2 copper layers, 85 x 56.5 mm, 104 parts, among them J1 RJ11, J2 2x20 0.1" Stacking Header, J3 8R, Q1 NPN 300V 0.5A, Q2 PNP 300V 0.5A, Q3 NPN 300V 0.5A, Q4 NPN 80V 330mW, Q5 NPN 80V 330mW, SW1 SW_SPDT, U1 Si2457-D-FT, U2 Si3018-F-GS, U3 74LVC541, U4 LM4819, U5 24LC32, U6 25LC320, Y1 32.768kHz 25ppm

Commit message: added more mfg part numbers
Parts:
- U1: value Si2457-D-FT -> Si2457
- U2: value Si3018-F-GS -> Si3018
Changed lines of the file:
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@@
     (descr "SMD package TO-269AA (e.g. diode bridge), see http://www.vishay.com/docs/88854/padlayouts.pdf")
     (tags "TO-269AA MBS diode bridge")
-    (property "MPN" "MB4S")
+    (property "MPN" "MB4S-TP")
     (property "Sheetfile" "ModemHAT.kicad_sch")
     (property "Sheetname" "")
@@
     (descr "http://www.onsemi.com/pub/Collateral/510CD.PDF")
     (tags "WQFN-20 4.5mm 2.5mm 0.5mm")
+    (property "MPN" "74LVC541ABQ,115")
     (property "Sheetfile" "ModemHAT.kicad_sch")
     (property "Sheetname" "")
@@
     (descr "TSSOP, 24 Pin (JEDEC MO-153 Var AD https://www.jedec.org/document_search?search_api_views_fulltext=MO-153), generated with kicad-footprint-generator ipc_gullwing_generator.py")
     (tags "TSSOP SO")
+    (property "MPN" "Si2457-D-FT")
     (property "Sheetfile" "ModemHAT.kicad_sch")
     (property "Sheetname" "")
@@
       (effects (font (size 1 1) (thickness 0.15)))
     )
-    (fp_text value "Si2457-D-FT" (at 0 4.85) (layer "F.Fab")
+    (fp_text value "Si2457" (at 0 4.85) (layer "F.Fab")
       (effects (font (size 1 1) (thickness 0.15)))
     )
@@
     (descr "Capacitor SMD 0805 (2012 Metric), square (rectangular) end terminal, IPC_7351 nominal, (Body size source: IPC-SM-782 page 76, https://www.pcb-3d.com/wordpress/wp-content/uploads/ipc-sm-782a_amendment_1_and_2.pdf, https://docs.google.com/spreadsheets/d/1BsfQQcO9C6DZCsRaXUlFlo91Tg2WpOkGARC1WS5S8t0/edit?usp=sharing), generated with kicad-footprint-generator")
     (tags "capacitor")
+    (property "MPN" "GRM21BR72E103KW03L")
     (property "Sheetfile" "ModemHAT.kicad_sch")
     (property "Sheetname" "")
@@
     (descr "Sub-miniature slide switch, right-angle, http://www.ckswitches.com/media/1422/js.pdf")
     (tags "switch spdt")
+    (property "MPN" "JS102011SAQN")
     (property "Sheetfile" "ModemHAT.kicad_sch")
     (property "Sheetname" "")
@@
     (property "Sheetfile" "ModemHAT.kicad_sch")
     (property "Sheetname" "")
-    (attr exclude_from_pos_files)
+    (property "exclude_from_bom" "")
+    (attr exclude_from_pos_files exclude_from_bom)
     (fp_text reference "H3" (at 0 -3.7) (layer "F.SilkS") hide
       (effects (font (size 1 1) (thickness 0.15)))
@@
     (descr "Capacitor SMD 1812 (4532 Metric), square (rectangular) end terminal, IPC_7351 nominal, (Body size source: IPC-SM-782 page 76, https://www.pcb-3d.com/wordpress/wp-content/uploads/ipc-sm-782a_amendment_1_and_2.pdf), generated with kicad-footprint-generator")
     (tags "capacitor")
+    (property "MPN" "502R29W681KV3E-****-SC")
     (property "Sheetfile" "ModemHAT.kicad_sch")
     (property "Sheetname" "")
@@
     (descr "RJ12 connector  https://cdn.amphenol-icc.com/media/wysiwyg/files/drawing/c-bmj-0082.pdf")
     (tags "RJ12 connector")
+    (property "MPN" "54601-906001WPLF")
     (property "Sheetfile" "ModemHAT.kicad_sch")
     (property "Sheetname" "")
@@
     (descr "Capacitor SMD 1812 (4532 Metric), square (rectangular) end terminal, IPC_7351 nominal, (Body size source: IPC-SM-782 page 76, https://www.pcb-3d.com/wordpress/wp-content/uploads/ipc-sm-782a_amendment_1_and_2.pdf), generated with kicad-footprint-generator")
     (tags "capacitor")
+    (property "MPN" "502R29W681KV3E-****-SC")
     (property "Sheetfile" "ModemHAT.kicad_sch")
     (property "Sheetname" "")
@@
     (property "Sheetfile" "ModemHAT.kicad_sch")
     (property "Sheetname" "")
-    (attr exclude_from_pos_files)
+    (property "exclude_from_bom" "")
+    (attr exclude_from_pos_files exclude_from_bom)
     (fp_text reference "H1" (at 0 -3.7) (layer "F.SilkS") hide
       (effects (font (size 1 1) (thickness 0.15)))
@@
     (descr "SOIC, 16 Pin (JEDEC MS-012AC, https://www.analog.com/media/en/package-pcb-resources/package/pkg_pdf/soic_narrow-r/r_16.pdf), generated with kicad-footprint-generator ipc_gullwing_generator.py")
     (tags "SOIC SO")
+    (property "MPN" "Si3018-F-GS")
     (property "Sheetfile" "ModemHAT.kicad_sch")
     (property "Sheetname" "")
@@
       (effects (font (size 1 1) (thickness 0.15)))
     )
-    (fp_text value "Si3018-F-GS" (at 0 5.9) (layer "F.Fab")
+    (fp_text value "Si3018" (at 0 5.9) (layer "F.Fab")
       (effects (font (size 1 1) (thickness 0.15)))
     )
@@
     (descr "TSSOP, 8 Pin (JEDEC MO-153 Var AA https://www.jedec.org/document_search?search_api_views_fulltext=MO-153), generated with kicad-footprint-generator ipc_gullwing_generator.py")
     (tags "TSSOP SO")
+    (property "MPN" "CAT24C32YI-GT3")
     (property "Sheetfile" "ModemHAT.kicad_sch")
     (property "Sheetname" "")
@@
     (descr "TSSOP, 8 Pin (JEDEC MO-153 Var AA https://www.jedec.org/document_search?search_api_views_fulltext=MO-153), generated with kicad-footprint-generator ipc_gullwing_generator.py")
     (tags "TSSOP SO")
+    (property "MPN" "25LC320AT-I/ST")
     (property "Sheetfile" "ModemHAT.kicad_sch")
     (property "Sheetname" "")
@@
     (descr "SOIC, 8 Pin (JEDEC MS-012AA, https://www.analog.com/media/en/package-pcb-resources/package/pkg_pdf/soic_narrow-r/r_8.pdf), generated with kicad-footprint-generator ipc_gullwing_generator.py")
     (tags "SOIC SO")
+    (property "MPN" "LM4819MX/NOPB")
     (property "Sheetfile" "ModemHAT.kicad_sch")
     (property "Sheetname" "")
@@
     (property "Sheetfile" "ModemHAT.kicad_sch")
     (property "Sheetname" "")
-    (attr exclude_from_pos_files)
+    (property "exclude_from_bom" "")
+    (attr exclude_from_pos_files exclude_from_bom)
     (fp_text reference "H2" (at 0 -3.7) (layer "F.SilkS") hide
       (effects (font (size 1 1) (thickness 0.15)))
@@
     (property "Sheetfile" "ModemHAT.kicad_sch")
     (property "Sheetname" "")
-    (attr exclude_from_pos_files)
+    (property "exclude_from_bom" "")
+    (attr exclude_from_pos_files exclude_from_bom)
     (fp_text reference "H4" (at 0 -3.7) (layer "F.SilkS") hide
       (effects (font (size 1 1) (thickness 0.15)))
