File: ModemHAT.kicad_pcb (KiCad board)
At the start: 2 copper layers, 85 x 56.5 mm, 104 parts, among them J1 RJ11, J2 2x20 0.1" Stacking Header, J3 8R, Q1 NPN 300V 0.5A, Q2 PNP 300V 0.5A, Q3 NPN 300V 0.5A, Q4 NPN 80V 330mW, Q5 NPN 80V 330mW, SW1 SW_SPDT, U1 Si2457, U2 Si3018, U3 74LVC541, U4 LM4819, U5 24LC32, U6 25LC320, Y1 32.768kHz 25ppm

Commit message: rev B
Parts:
- removed RN1, RN2: 470R, Resistor_SMD:R_Array_Concave_4x0603
- removed kibuzzard-6270B766: G***, kibuzzard-6270B766
- removed kibuzzard-6270B7C1: G***, kibuzzard-6270B7C1
- added LS1: Speaker, Buzzer_Beeper:Buzzer_15x7.5RM7.6, F.Cu at (90.8, 102.3)
- added R34: 1K, Resistor_SMD:R_0603_1608Metric, F.Cu at (123.5, 112.8)
- added R35: 1K, Resistor_SMD:R_0603_1608Metric, F.Cu at (120.3, 112.8)
- added R36: 1K, Resistor_SMD:R_0603_1608Metric, F.Cu at (117.1, 112.8)
- added R37: 1K, Resistor_SMD:R_0603_1608Metric, F.Cu at (113.9, 112.8)
- added R38: 1K, Resistor_SMD:R_0603_1608Metric, F.Cu at (110.8, 112.8)
- added R39: 1K, Resistor_SMD:R_0603_1608Metric, F.Cu at (107.6, 112.8)
- added R40: 1K, Resistor_SMD:R_0603_1608Metric, F.Cu at (104.4, 112.8)
- added R41: 1K, Resistor_SMD:R_0603_1608Metric, F.Cu at (101.2, 112.8)
- added kibuzzard-665D11B2: G***, kibuzzard-665D11B2, F.Cu at (83.6, 111.1)
- added kibuzzard-665D1212: G***, kibuzzard-665D1212, F.Cu at (87.6, 117.5)
- C3: value 10nF 250V -> 0.01uF 250V
- J1: footprint Connector_RJ:RJ12_Amphenol_54601 -> Connector_RJ:RJ12_Amphenol_54601-x06_Horizontal
- J3: value 8R -> JST
- R1, R11: footprint Resistor_SMD:R_2010_5025Metric -> Resistor_SMD:R_1210_3225Metric
- R18: value DNP -> 10K
- R26: value 200R -> 150R
- R29, R30, R31, R32: value DNP -> 0R
- R4: footprint Resistor_SMD:R_1206_3216Metric -> Resistor_SMD:R_1210_3225Metric
- SW1: footprint Button_Switch_SMD:SW_SPDT_CK-JS102011SAQN -> Button_Switch_SMD:SW_SPDT_CK_JS102011SAQN
- U3: footprint Package_DFN_QFN:WQFN-20-1EP_2.5x4.5mm_P0.5mm_EP1x2.9mm -> Package_SO:TSSOP-20_4.4x6.5mm_P0.65mm
- moved R24 7.26 mm to (88.4, 91.9), turned to -90 degrees
- moved C12 6.18 mm to (86.9, 91.9), turned to -90 degrees
- moved U3 3.33 mm to (109.0, 105.7)
- moved C11 2.22 mm to (113.4, 107.8)
- moved C7 1.60 mm to (131.9, 89.0)
- moved U4 1.41 mm to (91.9, 91.8)
- moved C13 1.36 mm to (91.9, 96.3)
- moved R17 1.31 mm to (113.4, 103.6), turned to 90 degrees
- moved C14 1.30 mm to (92.3, 81.6)
- moved C16 1.30 mm to (87.8, 81.6)
- moved C18 1.30 mm to (93.9, 84.6)
- moved R19 1.30 mm to (93.8, 81.6)
- moved C15 1.30 mm to (91.7, 85.4)
- moved C17 1.30 mm to (88.7, 83.9)
- moved C19 1.30 mm to (91.7, 86.9)
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Routing:
- net /SPKR-: track 17.7 -> 27.3 mm
- net /SPKR+: track 14.0 -> 21.8 mm
- net Net-(U3-Y0): track 7.36 -> 14.9 mm
- net Net-(U3-Y1): track 7.29 -> 12.4 mm
- net GND: track 48.0 -> 52.9 mm, vias 123 -> 124
- net /~{DCD}: track 16.9 -> 12.4 mm
- net /UART4_CTS: track 51.6 -> 47.3 mm
- net Net-(D2-K): track 5.83 -> 1.55 mm
- net /TXD: track 60.0 -> 55.8 mm
- net /RXD: track 53.0 -> 48.8 mm
- net /UART4_RTS: track 54.4 -> 50.3 mm
- net Net-(U4--IN): track 11.2 -> 7.16 mm
- net /MUTE: track 25.4 -> 29.1 mm
- net Net-(D9-K): track 4.86 -> 1.54 mm
- net Net-(D6-K): track 4.66 -> 1.56 mm
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Other:
- board text removed: "Speaker"
